Commit message: Add camera to robot

File: urdf/my_robot.xacro (robot description, xacro)
@@ -119,3 +119,33 @@
     <dynamics damping="1.0" friction="1.0"/>
   </joint>
+  <link name="camera">
+    <inertial>
+      <mass value="0.1"/>
+      <origin xyz="0 0 0"/>
+      <box_inertia m="0.1" x="0.05" y="0.05" z="0.05">
+      <inertia
+          ixx="1e-6" ixy="0" ixz="0"
+          iyy="1e-6" iyz="0"
+          izz="1e-6"
+      />
+    </inertial>
+    <collision name='camera_collision'>
+      <origin xyz="0 0 0" rpy="0 0 0"/>
+      <geometry>
+        <box size="0.05 0.05 0.05"/>
+      </geometry>
+    </collision>
+    <visual name='camera_visual'>
+      <origin xyz="0 0 0" rpy="0 0 0"/>
+      <geometry>
+        <box size="0.05 0.05 0.05"/>
+      </geometry>
+    </visual>
+  </link>
+  <joint type="fixed" name="camera_joint">
+    <origin xyz="0.2 0 0" rpy="0 0 0"/>
+    <child link="camera"/>
+    <parent link="chassis"/>
+    <axis xyz="0 1 0" rpy="0 0 0"/>
+  </joint>
 </robot>

Commit message: Adds lidar to robot model

File: urdf/my_robot.xacro (robot description, xacro)
@@ -149,3 +149,33 @@
     <axis xyz="0 1 0" rpy="0 0 0"/>
   </joint>
+  <link name="hokuyo">
+    <inertial>
+      <mass value="1e-5">
+      <origin xyz="0 0 0" rpy="0 0 0"/>
+      <box_inertia m="0.1" x="0.05" y="0.05" z="0.05">
+      <inertia
+          ixx="1e-6" ixy="0" ixz="0"
+          iyy="1e-6" iyz="0"
+          izz="1e-6"
+      />
+    </inertial>
+    <collision name='hokuyo_collision'>
+      <origin xyz="0 0 0" rpy="0 0 0"/>
+      <geometry>
+        <box size="0.1 0.1 0.1"/>
+      </geometry>
+    </collision>
+    <visual name='hokuyo_visual'>
+      <origin xyz="0 0 0" rpy="0 0 0"/>
+      <geometry>
+        <filename="package://my_robot/meshes/hokuyo.dae"/>
+      </geometry>
+    </visual>
+  </link>
+  <joint type="fixed" name="hokuyo_joint">
+    <origin xyz="0.15 0 0.1" rpy="0 0 0"/>
+    <child link="hokuyo"/>
+    <parent link="chassis"/>
+    <axis xyz="0 1 0" rpy="0 0 0"/>
+  </joint>
 </robot>

Commit message: robot model - experiment with colours/material

File: urdf/my_robot.xacro (robot description, xacro)
@@ -119,4 +119,7 @@
     <dynamics damping="1.0" friction="1.0"/>
   </joint>
+  <gazebo reference="left_wheel">
+      <material>Gazebo/Green</material>
+  </gazebo>
   <link name="camera">
     <inertial>

Commit message: fix xml
fix xml

fix xml

fix xml

fix xml

File: urdf/my_robot.xacro (robot description, xacro)
@@ -126,5 +126,5 @@
       <mass value="0.1"/>
       <origin xyz="0 0 0"/>
-      <box_inertia m="0.1" x="0.05" y="0.05" z="0.05">
+      <box_inertia m="0.1" x="0.05" y="0.05" z="0.05"/>
       <inertia
           ixx="1e-6" ixy="0" ixz="0"
@@ -154,7 +154,6 @@
   <link name="hokuyo">
     <inertial>
-      <mass value="1e-5">
+      <mass value="1e-5"/>
       <origin xyz="0 0 0" rpy="0 0 0"/>
-      <box_inertia m="0.1" x="0.05" y="0.05" z="0.05">
       <inertia
           ixx="1e-6" ixy="0" ixz="0"
@@ -172,5 +171,5 @@
       <origin xyz="0 0 0" rpy="0 0 0"/>
       <geometry>
-        <filename="package://my_robot/meshes/hokuyo.dae"/>
+        <mesh filename="package://my_robot/meshes/hokuyo.dae"/>
       </geometry>
     </visual>

Commit message: fix xml

File: urdf/my_robot.xacro (robot description, xacro)
@@ -154,5 +154,5 @@
   <link name="hokuyo">
     <inertial>
-      <mass value="1e-5">
+      <mass value="1e-5"/>
       <origin xyz="0 0 0" rpy="0 0 0"/>
       <inertia

Commit message: fix xml

File: urdf/my_robot.xacro (robot description, xacro)
@@ -170,7 +170,5 @@
     <visual name='hokuyo_visual'>
       <origin xyz="0 0 0" rpy="0 0 0"/>
-      <geometry>
-        <filename="package://my_robot/meshes/hokuyo.dae"/>
-      </geometry>
+      <geometry filename="package://my_robot/meshes/hokuyo.dae"/>
     </visual>
   </link>

Commit message: fix xml

File: urdf/my_robot.xacro (robot description, xacro)
@@ -170,5 +170,7 @@
     <visual name='hokuyo_visual'>
       <origin xyz="0 0 0" rpy="0 0 0"/>
-      <geometry filename="package://my_robot/meshes/hokuyo.dae"/>
+      <geometry>
+        <mesh filename="package://my_robot/meshes/hokuyo.dae"/>
+      </geometry>
     </visual>
   </link>

Commit message: Adding plugin to my_robot for control

File: urdf/my_robot.xacro (robot description, xacro)
@@ -1,4 +1,5 @@
 <?xml version='1.0'?>
 <robot name="my_robot" xmlns:xacro="http://www.ros.org/wiki/xacro">
+  <xacro:include filename="$(find my_robot)/urdf/my_robot.gazebo" />
   <link name="robot_footprint"></link>
   <joint name="robot_footprint_joint" type="fixed">
@@ -119,7 +120,4 @@
     <dynamics damping="1.0" friction="1.0"/>
   </joint>
-  <gazebo reference="left_wheel">
-      <material>Gazebo/Green</material>
-  </gazebo>
   <link name="camera">
     <inertial>
@@ -181,3 +179,12 @@
     <axis xyz="0 1 0" rpy="0 0 0"/>
   </joint>
+  <gazebo reference="left_wheel">
+      <material>Gazebo/Blue</material>
+  </gazebo>
+  <gazebo reference="right_wheel">
+      <material>Gazebo/Blue</material>
+  </gazebo>
+  <gazebo reference="camera">
+      <material>Gazebo/Black</material>
+  </gazebo>
 </robot>
